Commit message: Add wheels to robot

File: src/my_robot/urdf/my_robot.xacro (robot description, xacro)
@@ -55,3 +55,65 @@
         </visual>
     </link>
+    <link name="left_wheel">
+        <inertial>
+            <mass value="5.0"/>
+            <origin xyz="0 0 0" rpy="0 0 0"/>
+            <inertia
+                ixx="0.1" ixy="0"   ixz="0"
+                          iyy="0.1" iyz="0"
+                                    izz="0.1"
+            />
+        </inertial>
+        <collision name="left_wheel_collision">
+            <origin xyz="0 0 0" rpy="0 1.5707 1.5707"/>
+            <geometry>
+                <cylinder radius="0.1" length="0.05"/>
+            </geometry>
+        </collision>
+        <visual name="left_wheel_visual">
+            <origin xyz="0 0 0" rpy="0 1.5707 1.5707"/>
+            <geometry>
+                <cylinder radius="0.1" length="0.05"/>
+            </geometry>
+        </visual>
+    </link>
+    <link name="right_wheel">
+        <inertial>
+            <mass value="5.0"/>
+            <origin xyz="0 0 0" rpy="0 0 0"/>
+            <inertia
+                ixx="0.1" ixy="0"   ixz="0"
+                          iyy="0.1" iyz="0"
+                                    izz="0.1"
+            />
+        </inertial>
+        <collision name="right_wheel_collision">
+            <origin xyz="0 0 0" rpy="0 1.5707 1.5707"/>
+            <geometry>
+                <cylinder radius="0.1" length="0.05"/>
+            </geometry>
+        </collision>
+        <visual name="right_wheel_visual">
+            <origin xyz="0 0 0" rpy="0 1.5707 1.5707"/>
+            <geometry>
+                <cylinder radius="0.1" length="0.05"/>
+            </geometry>
+        </visual>
+    </link>
+    <joint type="continuous" name="left_wheel_hinge">
+        <origin xyz="0 0.125 0" rpy="0 0 0"/>
+        <child link="left_wheel"/>
+        <parent link="chassis"/>
+        <axis xyz="0 1 0" rpy="0 0 0"/>
+        <limit effort="10000" velocity="1000"/>
+        <dynamics damping="1.0" friction="1.0"/>
+    </joint>
+    <joint type="continuous" name="right_wheel_hinge">
+        <origin xyz="0 -0.125 0" rpy="0 0 0"/>
+        <child link="right_wheel"/>
+        <parent link="chassis"/>
+        <axis xyz="0 1 0" rpy="0 0 0"/>
+        <limit effort="10000" velocity="1000"/>
+        <dynamics damping="1.0" friction="1.0"/>
+    </joint>
 </robot>

Commit message: Personalised differential drive robot
Now it is a two wheeled roomba-like robot

File: src/my_robot/urdf/my_robot.xacro (robot description, xacro)
@@ -1,119 +1,109 @@
 <?xml version="1.0"?>
 <robot name="my_robot" xmlns:xacro="http://www.ros.org/wiki/xacro">
+    <!-- CONSTANTS -->
+    <xacro:property name="pi" value="3.1415926535897931" />
+    <!-- Multiplicative factor applied to the radius of the caster balls
+         for them not to stop both wheels to be touching the ground at
+         the same time                                               -->
+    <xacro:property name="reduction_factor_caster_radius" value="0.998" />
+    <!-- PARAMETERS -->
+    <xacro:property name="wheel_radius" value="0.1" />
+    <xacro:property name="wheel_length" value="0.05" />
+    <xacro:property name="wheel_mass" value="5.0" />
+    <xacro:property name="base_radius" value="0.4" />
+    <xacro:property name="base_height" value="0.1" />
+    <xacro:property name="base_mass" value="15.0" />
+    <!-- MACROS -->
+    <!-- Inertial of a cylinder -->
+    <xacro:macro name="cylinder_inertial" params="mass radius length">
+        <inertial>
+            <mass value="${mass}" />
+            <inertia
+                ixx="${1/12*mass*(3*radius*radius + length*length)}" ixy="0" ixz="0"
+                iyy="${1/12*mass*(3*radius*radius + length*length)}" iyz="0"
+                izz="${1/2*mass*radius*radius}"
+            />
+        </inertial>
+    </xacro:macro>
+    <!-- Add a wheel and its joint on the x axis, outer part of the base -->
+    <xacro:macro name="wheel" params="side reflect">
+        <link name="${side}_wheel">
+            <xacro:cylinder_inertial
+                mass="${wheel_mass}" radius="${wheel_radius}" length="${wheel_length}"
+            />
+            <collision name="${side}_wheel_collision">
+                <origin xyz="0 0 0" rpy="0 ${pi/2} ${pi/2}"/>
+                <geometry>
+                    <cylinder radius="${wheel_radius}" length="${wheel_length}"/>
+                </geometry>
+            </collision>
+            <visual name="${side}_wheel_visual">
+                <origin xyz="0 0 0" rpy="0 ${pi/2} ${pi/2}"/>
+                <geometry>
+                    <cylinder radius="${wheel_radius}" length="${wheel_length}"/>
+                </geometry>
+            </visual>
+        </link>
+        <joint type="continuous" name="${side}_wheel_hinge">
+            <origin xyz="0 ${reflect*(base_radius + wheel_length/2)} 0" rpy="0 0 0"/>
+            <child link="${side}_wheel"/>
+            <parent link="base"/>
+            <axis xyz="0 1 0" rpy="0 0 0"/>
+            <limit effort="10000" velocity="1000"/>
+            <dynamics damping="1.0" friction="1.0"/>
+        </joint>
+    </xacro:macro>
+    <!-- ROBOT -->
     <link name="robot_footprint"></link>
     <joint name="robot_footprint_joint" type="fixed">
         <origin xyz="0 0 0" rpy="0 0 0"/>
         <parent link="robot_footprint"/>
-        <child link="chassis"/>
+        <child link="base"/>
     </joint>
-    <link name="chassis">
-        <pose>0 0 0.1 0 0 0</pose>
-        <inertial>
-            <mass value="15.0"/>
-            <origin xyz="0 0 0" rpy="0 0 0"/>
-            <inertia
-                ixx="0.1" ixy="0"   ixz="0"
-                          iyy="0.1" iyz="0"
-                                    izz="0.1"
-            />
-        </inertial>
-        <collision name="collision">
+    <!-- Cylindrical base with two casters for stability along the y axis-->
+    <link name="base">
+        <pose>0 0 ${wheel_radius} 0 0 0</pose>
+        <xacro:cylinder_inertial
+            mass="${base_mass}" radius="${base_radius}" length="${base_height}"
+        />
+        <collision name="base_collision">
             <origin xyz="0 0 0" rpy="0 0 0"/>
             <geometry>
-                <box size="0.4 0.2 0.1"/>
+                <cylinder radius="${base_radius}" length="${base_height}" />
             </geometry>
         </collision>
-        <visual name="chassis_visual">
+        <visual name="base_visual">
             <origin xyz="0 0 0" rpy="0 0 0"/>
             <geometry>
-                <box size="0.4 0.2 0.1"/>
+                <cylinder radius="${base_radius}" length="${base_height}" />
             </geometry>
         </visual>
         <collision name="back_caster_collision">
-            <origin xyz="-0.15 0 -0.05" rpy="0 0 0"/>
+            <origin xyz="${-3/4*base_radius} 0 ${-wheel_radius/2}" rpy="0 0 0"/>
             <geometry>
-                <sphere radius="0.0499"/>
+                <sphere radius="${reduction_factor_caster_radius*wheel_radius/2}"/>
             </geometry>
         </collision>
         <visual name="back_caster_visual">
-            <origin xyz="-0.15 0 -0.05" rpy="0 0 0"/>
+            <origin xyz="${-3/4*base_radius} 0 ${-wheel_radius/2}" rpy="0 0 0"/>
             <geometry>
-                <sphere radius="0.05"/>
+                <sphere radius="${wheel_radius/2}"/>
             </geometry>
         </visual>
         <collision name="front_caster_collision">
-            <origin xyz="0.15 0 -0.05" rpy="0 0 0"/>
+            <origin xyz="${3/4*base_radius} 0 ${-wheel_radius/2}" rpy="0 0 0"/>
             <geometry>
-                <sphere radius="0.0499"/>
+                <sphere radius="${reduction_factor_caster_radius*wheel_radius/2}"/>
             </geometry>
         </collision>
         <visual name="front_caster_visual">
-            <origin xyz="0.15 0 -0.05" rpy="0 0 0"/>
+            <origin xyz="${3/4*base_radius} 0 ${-wheel_radius/2}" rpy="0 0 0"/>
             <geometry>
-                <sphere radius="0.05"/>
+                <sphere radius="${wheel_radius/2}"/>
             </geometry>
         </visual>
     </link>
-    <link name="left_wheel">
-        <inertial>
-            <mass value="5.0"/>
-            <origin xyz="0 0 0" rpy="0 0 0"/>
-            <inertia
-                ixx="0.1" ixy="0"   ixz="0"
-                          iyy="0.1" iyz="0"
-                                    izz="0.1"
-            />
-        </inertial>
-        <collision name="left_wheel_collision">
-            <origin xyz="0 0 0" rpy="0 1.5707 1.5707"/>
-            <geometry>
-                <cylinder radius="0.1" length="0.05"/>
-            </geometry>
-        </collision>
-        <visual name="left_wheel_visual">
-            <origin xyz="0 0 0" rpy="0 1.5707 1.5707"/>
-            <geometry>
-                <cylinder radius="0.1" length="0.05"/>
-            </geometry>
-        </visual>
-    </link>
-    <link name="right_wheel">
-        <inertial>
-            <mass value="5.0"/>
-            <origin xyz="0 0 0" rpy="0 0 0"/>
-            <inertia
-                ixx="0.1" ixy="0"   ixz="0"
-                          iyy="0.1" iyz="0"
-                                    izz="0.1"
-            />
-        </inertial>
-        <collision name="right_wheel_collision">
-            <origin xyz="0 0 0" rpy="0 1.5707 1.5707"/>
-            <geometry>
-                <cylinder radius="0.1" length="0.05"/>
-            </geometry>
-        </collision>
-        <visual name="right_wheel_visual">
-            <origin xyz="0 0 0" rpy="0 1.5707 1.5707"/>
-            <geometry>
-                <cylinder radius="0.1" length="0.05"/>
-            </geometry>
-        </visual>
-    </link>
-    <joint type="continuous" name="left_wheel_hinge">
-        <origin xyz="0 0.125 0" rpy="0 0 0"/>
-        <child link="left_wheel"/>
-        <parent link="chassis"/>
-        <axis xyz="0 1 0" rpy="0 0 0"/>
-        <limit effort="10000" velocity="1000"/>
-        <dynamics damping="1.0" friction="1.0"/>
-    </joint>
-    <joint type="continuous" name="right_wheel_hinge">
-        <origin xyz="0 -0.125 0" rpy="0 0 0"/>
-        <child link="right_wheel"/>
-        <parent link="chassis"/>
-        <axis xyz="0 1 0" rpy="0 0 0"/>
-        <limit effort="10000" velocity="1000"/>
-        <dynamics damping="1.0" friction="1.0"/>
-    </joint>
+    <!-- Wheels on the x axis with their corresponding joints -->
+    <xacro:wheel side="left" reflect="-1" />
+    <xacro:wheel side="right" reflect="1" />
 </robot>

Commit message: Add rotating basis for the camera

File: src/my_robot/urdf/my_robot.xacro (robot description, xacro)
@@ -14,4 +14,6 @@
     <xacro:property name="base_height" value="0.1" />
     <xacro:property name="base_mass" value="15.0" />
+    <xacro:property name="camera_base_heigth" value="${(2*wheel_radius - base_height)/2}" />
+    <xacro:property name="camera_base_mass" value="5.0" />
     <!-- MACROS -->
     <!-- Inertial of a cylinder -->
@@ -107,3 +109,29 @@
     <xacro:wheel side="left" reflect="-1" />
     <xacro:wheel side="right" reflect="1" />
+    <!-- Rotating base for the camera -->
+    <link name="camera_base">
+        <xacro:cylinder_inertial
+            mass="${camera_base_mass}" radius="${base_radius}" length="${camera_base_heigth}"
+        />
+        <collision name="camera_base_collision">
+            <origin xyz="0 0 0" rpy="0 0 0"/>
+            <geometry>
+                <cylinder radius="${base_radius}" length="${camera_base_heigth}" />
+            </geometry>
+        </collision>
+        <visual name="camera_base_visual">
+            <origin xyz="0 0 0" rpy="0 0 0"/>
+            <geometry>
+                <cylinder radius="${base_radius}" length="${camera_base_heigth}" />
+            </geometry>
+        </visual>
+    </link>
+    <joint name="camera_base_hinge" type="continuous">
+        <origin xyz="0 0 ${1/2*base_height + 1/2*camera_base_heigth}" rpy="0 0 0" />
+        <child link="camera_base" />
+        <parent link="base" />
+        <axis xyz="0 0 1" rpy="0 0 0" />
+        <limit effort="10000" velocity="1000" />
+        <dynamics damping="1.0" friction="1.0" />
+    </joint>
 </robot>

Commit message: Correct dimensions of base so that camera won't collide with wheels
Also, correct height of wheel joints

File: src/my_robot/urdf/my_robot.xacro (robot description, xacro)
@@ -7,13 +7,22 @@
          the same time                                               -->
     <xacro:property name="reduction_factor_caster_radius" value="0.998" />
+    <!-- </CONSTANTS> -->
     <!-- PARAMETERS -->
+    <!-- Base parameters -->
+    <xacro:property name="base_radius" value="0.4" />
+    <!-- base height must be inside (wheel_radius, 2*wheel_radius) -->
+    <!-- note that the extremes of the interval are not included   -->
+    <xacro:property name="base_height" value="0.15" />
+    <xacro:property name="base_mass" value="15.0" />
+    <!-- Wheel parameters -->
     <xacro:property name="wheel_radius" value="0.1" />
     <xacro:property name="wheel_length" value="0.05" />
     <xacro:property name="wheel_mass" value="5.0" />
-    <xacro:property name="base_radius" value="0.4" />
-    <xacro:property name="base_height" value="0.1" />
-    <xacro:property name="base_mass" value="15.0" />
-    <xacro:property name="camera_base_heigth" value="${(2*wheel_radius - base_height)/2}" />
-    <xacro:property name="camera_base_mass" value="5.0" />
+    <xacro:property name="z_offset_between_centers" value="${wheel_radius - base_height/2}" />
+    <!-- Sensor's base parameters -->
+    <xacro:property name="sensors_base_heigth" value="${(2*wheel_radius - base_height)/2}" />
+    <xacro:property name="sensors_base_mass" value="5.0" />
+    <xacro:property name="sensors_base_offset_z" value="${base_height/2 + sensors_base_heigth/2}" />
+    <!-- </PARAMETERS> -->
     <!-- MACROS -->
     <!-- Inertial of a cylinder -->
@@ -48,5 +57,8 @@
         </link>
         <joint type="continuous" name="${side}_wheel_hinge">
-            <origin xyz="0 ${reflect*(base_radius + wheel_length/2)} 0" rpy="0 0 0"/>
+            <origin
+                xyz="0 ${reflect*(base_radius + wheel_length/2)} ${-z_offset_between_centers}"
+                rpy="0 0 0"
+            />
             <child link="${side}_wheel"/>
             <parent link="base"/>
@@ -56,5 +68,6 @@
         </joint>
     </xacro:macro>
-    <!-- ROBOT -->
+    <!-- </MACROS> -->
+    <!-- ROBOT DESCRIPTION-->
     <link name="robot_footprint"></link>
     <joint name="robot_footprint_joint" type="fixed">
@@ -65,5 +78,7 @@
     <!-- Cylindrical base with two casters for stability along the y axis-->
     <link name="base">
-        <pose>0 0 ${wheel_radius} 0 0 0</pose>
+        <!-- we want the wheel to touch the ground and the top of the base
+             to coincide with the top of the wheel                       -->
+        <pose>0 0 ${wheel_radius + z_offset_between_centers} 0 0 0</pose>
         <xacro:cylinder_inertial
             mass="${base_mass}" radius="${base_radius}" length="${base_height}"
@@ -82,5 +97,8 @@
         </visual>
         <collision name="back_caster_collision">
-            <origin xyz="${-3/4*base_radius} 0 ${-wheel_radius/2}" rpy="0 0 0"/>
+            <origin
+                xyz="${-3/4*base_radius} 0 ${-wheel_radius/2 - z_offset_between_centers}"
+                rpy="0 0 0"
+            />
             <geometry>
                 <sphere radius="${reduction_factor_caster_radius*wheel_radius/2}"/>
@@ -88,5 +106,8 @@
         </collision>
         <visual name="back_caster_visual">
-            <origin xyz="${-3/4*base_radius} 0 ${-wheel_radius/2}" rpy="0 0 0"/>
+            <origin
+                xyz="${-3/4*base_radius} 0 ${-wheel_radius/2 - z_offset_between_centers}"
+                rpy="0 0 0"
+            />
             <geometry>
                 <sphere radius="${wheel_radius/2}"/>
@@ -94,5 +115,8 @@
         </visual>
         <collision name="front_caster_collision">
-            <origin xyz="${3/4*base_radius} 0 ${-wheel_radius/2}" rpy="0 0 0"/>
+            <origin
+                xyz="${3/4*base_radius} 0 ${-wheel_radius/2 - z_offset_between_centers}"
+                rpy="0 0 0"
+            />
             <geometry>
                 <sphere radius="${reduction_factor_caster_radius*wheel_radius/2}"/>
@@ -100,5 +124,8 @@
         </collision>
         <visual name="front_caster_visual">
-            <origin xyz="${3/4*base_radius} 0 ${-wheel_radius/2}" rpy="0 0 0"/>
+            <origin
+                xyz="${3/4*base_radius} 0 ${-wheel_radius/2 - z_offset_between_centers}"
+                rpy="0 0 0"
+            />
             <geometry>
                 <sphere radius="${wheel_radius/2}"/>
@@ -109,25 +136,25 @@
     <xacro:wheel side="left" reflect="-1" />
     <xacro:wheel side="right" reflect="1" />
-    <!-- Rotating base for the camera -->
-    <link name="camera_base">
+    <!-- Rotating base for the sensors -->
+    <link name="sensors_base">
         <xacro:cylinder_inertial
-            mass="${camera_base_mass}" radius="${base_radius}" length="${camera_base_heigth}"
+            mass="${sensors_base_mass}" radius="${base_radius}" length="${sensors_base_heigth}"
         />
-        <collision name="camera_base_collision">
+        <collision name="sensors_base_collision">
             <origin xyz="0 0 0" rpy="0 0 0"/>
             <geometry>
-                <cylinder radius="${base_radius}" length="${camera_base_heigth}" />
+                <cylinder radius="${base_radius}" length="${sensors_base_heigth}" />
             </geometry>
         </collision>
-        <visual name="camera_base_visual">
+        <visual name="sensors_base_visual">
             <origin xyz="0 0 0" rpy="0 0 0"/>
             <geometry>
-                <cylinder radius="${base_radius}" length="${camera_base_heigth}" />
+                <cylinder radius="${base_radius}" length="${sensors_base_heigth}" />
             </geometry>
         </visual>
     </link>
-    <joint name="camera_base_hinge" type="continuous">
-        <origin xyz="0 0 ${1/2*base_height + 1/2*camera_base_heigth}" rpy="0 0 0" />
-        <child link="camera_base" />
+    <joint name="sensors_base_hinge" type="continuous">
+        <origin xyz="0 0 ${sensors_base_offset_z}" rpy="0 0 0" />
+        <child link="sensors_base" />
         <parent link="base" />
         <axis xyz="0 0 1" rpy="0 0 0" />
@@ -135,3 +162,4 @@
         <dynamics damping="1.0" friction="1.0" />
     </joint>
+    <!-- </ROBOT DESCRIPTION> -->
 </robot>

Commit message: Add camera

File: src/my_robot/urdf/my_robot.xacro (robot description, xacro)
@@ -20,6 +20,9 @@
     <xacro:property name="wheel_mass" value="5.0" />
     <xacro:property name="z_offset_between_centers" value="${wheel_radius - base_height/2}" />
+    <!-- Camera parameters -->
+    <xacro:property name="camera_edge_length" value="0.05" />
+    <xacro:property name="camera_mass" value="0.1" />
     <!-- Sensor's base parameters -->
-    <xacro:property name="sensors_base_heigth" value="${(2*wheel_radius - base_height)/2}" />
+    <xacro:property name="sensors_base_heigth" value="${1.5*camera_edge_length}" />
     <xacro:property name="sensors_base_mass" value="5.0" />
     <xacro:property name="sensors_base_offset_z" value="${base_height/2 + sensors_base_heigth/2}" />
@@ -34,4 +37,15 @@
                 iyy="${1/12*mass*(3*radius*radius + length*length)}" iyz="0"
                 izz="${1/2*mass*radius*radius}"
+            />
+        </inertial>
+    </xacro:macro>
+    <!-- Inertial of a cube -->
+    <xacro:macro name="cube_inertial" params="mass edge_length">
+        <inertial>
+            <mass value="${mass}" />
+            <inertia
+                ixx="${1/6*mass*edge_length*edge_length}" ixy="0" ixz="0"
+                iyy="${1/6*mass*edge_length*edge_length}" iyz="0"
+                izz="${1/6*mass*edge_length*edge_length}"
             />
         </inertial>
@@ -162,4 +176,26 @@
         <dynamics damping="1.0" friction="1.0" />
     </joint>
+    <!-- Camera -->
+    <link name="camera">
+        <xacro:cube_inertial mass="${camera_mass}" edge_length="${camera_edge_length}" />
+        <collision name="camera_collision">
+            <origin xyz="0 0 0" rpy="0 0 0" />
+            <geometry>
+                <box size="${camera_edge_length} ${camera_edge_length} ${camera_edge_length}" />
+            </geometry>
+        </collision>
+        <visual name="camera_visual">
+            <origin xyz="0 0 0" rpy="0 0 0" />
+            <geometry>
+                <box size="${camera_edge_length} ${camera_edge_length} ${camera_edge_length}" />
+            </geometry>
+        </visual>
+    </link>
+    <joint name="camera_joint" type="fixed">
+        <origin xyz="${base_radius} 0 0" rpy="0 0 0" />
+        <parent link="sensors_base" />
+        <child link="camera" />
+        <axis xyz="0 1 0" rpy="0 0 0" />
+    </joint>
     <!-- </ROBOT DESCRIPTION> -->
 </robot>

Commit message: Add hokuyo lidar

File: src/my_robot/urdf/my_robot.xacro (robot description, xacro)
@@ -23,4 +23,7 @@
     <xacro:property name="camera_edge_length" value="0.05" />
     <xacro:property name="camera_mass" value="0.1" />
+    <!-- Lidar parameters -->
+    <xacro:property name="lidar_edge_length" value="0.1" />
+    <xacro:property name="lidar_mass" value="1e-5" />
     <!-- Sensor's base parameters -->
     <xacro:property name="sensors_base_heigth" value="${1.5*camera_edge_length}" />
@@ -198,4 +201,29 @@
         <axis xyz="0 1 0" rpy="0 0 0" />
     </joint>
+    <!-- Lidar -->
+    <link name="hokuyo">
+        <xacro:cube_inertial mass="${lidar_mass}" edge_length="${lidar_edge_length}" />
+        <collision name="lidar_collision">
+            <origin xyz="0 0 0" rpy="0 0 0" />
+            <geometry>
+                <box size="${lidar_edge_length} ${lidar_edge_length} ${lidar_edge_length}" />
+            </geometry>
+        </collision>
+        <visual name="camera_visual">
+            <origin xyz="0 0 0" rpy="0 0 0" />
+            <geometry>
+                <mesh filename="package://my_robot/meshes/hokuyo.dae" />
+            </geometry>
+        </visual>
+    </link>
+    <joint name="hokuyo_joint" type="fixed">
+        <origin
+            xyz="${base_radius - lidar_edge_length} 0 ${sensors_base_heigth/2}"
+            rpy="0 0 0"
+        />
+        <parent link="sensors_base" />
+        <child link="hokuyo" />
+        <axis xyz="0 1 0" rpy="0 0 0" />
+    </joint>
     <!-- </ROBOT DESCRIPTION> -->
 </robot>
