Commit message: Correct format of first palette of colors

File: src/my_robot/urdf/materials.xacro (robot description, xacro)
@@ -3,19 +3,49 @@
     <!-- First palette -->
     <!-- https://coolors.co/fe938c-e6b89c-ead2ac-9cafb7-4281a4 -->
-    <material name="tulip">
-        <color rgba="${254/255} ${147/255} ${140/255} 1" />
-    </material>
-    <material name="pale_gold">
-        <color rgba="${230/255} ${184/255} ${156/255} 1" />
-    </material>
-    <material name="desert_sand">
-        <color rgba="${234/255} ${210/255} ${172/255} 1" />
-    </material>
-    <material name="pewter_blue">
-        <color rgba="${156/255} ${175/255} ${183/255} 1" />
-    </material>
-    <material name="steel_blue">
-        <color rgba="${66/255} ${129/255} ${164/255} 1" />
-    </material>
+    <xacro:macro name="material_tulip">
+        <visual>
+            <material>
+                <ambient>${254/255} ${147/255} ${140/255} 1</ambient>
+                <diffuse>${254/255} ${147/255} ${140/255} 1</diffuse>
+                <specular>0.1 0.1 0.1 0.1 1</specular>
+            </material>
+        </visual>
+    </xacro:macro>
+    <xacro:macro name="material_pale_gold">
+        <visual>
+            <material>
+                <ambient>${230/255} ${184/255} ${156/255} 1</ambient>
+                <diffuse>${230/255} ${184/255} ${156/255} 1</diffuse>
+                <specular>0.1 0.1 0.1 0.1 1</specular>
+            </material>
+        </visual>
+    </xacro:macro>
+    <xacro:macro name="material_desert_sand">
+        <visual>
+            <material>
+                <ambient>${234/255} ${210/255} ${172/255} 1</ambient>
+                <diffuse>${234/255} ${210/255} ${172/255} 1</diffuse>
+                <specular>0.1 0.1 0.1 0.1 1</specular>
+            </material>
+        </visual>
+    </xacro:macro>
+    <xacro:macro name="material_pewter_blue">
+        <visual>
+            <material>
+                <ambient>${156/255} ${175/255} ${183/255} 1</ambient>
+                <diffuse>${156/255} ${175/255} ${183/255} 1</diffuse>
+                <specular>0.1 0.1 0.1 0.1 1</specular>
+            </material>
+        </visual>
+    </xacro:macro>
+    <xacro:macro name="material_steel_blue">
+        <visual>
+            <material>
+                <ambient>${66/255} ${129/255} ${164/255} 1</ambient>
+                <diffuse>${66/255} ${129/255} ${164/255} 1</diffuse>
+                <specular>0.1 0.1 0.1 0.1 1</specular>
+            </material>
+        </visual>
+    </xacro:macro>
     <!-- Second palette -->
     <!-- https://coolors.co/5bc0eb-fde74c-9bc53d-e55934-fa7921 -->
